File: gpstracker-interface.sch (KiCad schematic (older format))
At the start: 13 parts, among them J1 USB_B_Micro, U6 FT231XS

Commit message: Started routing
Parts:
- J1: value USB_B_Micro -> Molex 47346-0001
Changed lines of the file:
@@
 $EndComp
 $Comp
-L +3.3V_FDTI #PWR51
+L +3.3V_FDTI #PWR047
 U 1 1 5A36BE13
 P 4450 1750
-F 0 "#PWR51" H 4450 1600 50  0001 C CNN
+F 0 "#PWR047" H 4450 1600 50  0001 C CNN
 F 1 "+3.3V_FDTI" H 4450 1890 50  0000 C CNN
 F 2 "" H 4450 1750 50  0001 C CNN
@@
 $EndComp
 $Comp
-L +3.3V_FDTI #PWR47
+L +3.3V_FDTI #PWR048
 U 1 1 5A36BE45
 P 2050 1650
-F 0 "#PWR47" H 2050 1500 50  0001 C CNN
+F 0 "#PWR048" H 2050 1500 50  0001 C CNN
 F 1 "+3.3V_FDTI" H 2050 1790 50  0000 C CNN
 F 2 "" H 2050 1650 50  0001 C CNN
@@
 $EndComp
 $Comp
-L GND #PWR46
+L GND #PWR049
 U 1 1 5A36E473
 P 2000 2700
-F 0 "#PWR46" H 2000 2450 50  0001 C CNN
+F 0 "#PWR049" H 2000 2450 50  0001 C CNN
 F 1 "GND" H 2000 2550 50  0000 C CNN
 F 2 "" H 2000 2700 50  0001 C CNN
@@
 $EndComp
 $Comp
-L GND #PWR49
+L GND #PWR050
 U 1 1 5A36E4AC
 P 2800 3300
-F 0 "#PWR49" H 2800 3050 50  0001 C CNN
+F 0 "#PWR050" H 2800 3050 50  0001 C CNN
 F 1 "GND" H 2800 3150 50  0000 C CNN
 F 2 "" H 2800 3300 50  0001 C CNN
@@
 P 1100 1000
 F 0 "J1" H 900 1450 50  0000 L CNN
-F 1 "USB_B_Micro" H 900 1350 50  0000 L CNN
+F 1 "Molex 47346-0001" H 900 1350 50  0001 L CNN
 F 2 "Connectors_USB:USB_Micro-B_Molex_47346-0001" H 1250 950 50  0001 C CNN
 F 3 "" H 1250 950 50  0001 C CNN
@@
 $EndComp
 $Comp
-L GND #PWR44
+L GND #PWR051
 U 1 1 5A36EE8C
 P 1350 2550
-F 0 "#PWR44" H 1350 2300 50  0001 C CNN
+F 0 "#PWR051" H 1350 2300 50  0001 C CNN
 F 1 "GND" H 1350 2400 50  0000 C CNN
 F 2 "" H 1350 2550 50  0001 C CNN
@@
 $EndComp
 $Comp
-L VBUS #PWR45
+L VBUS #PWR052
 U 1 1 5A36EF48
 P 1700 1000
-F 0 "#PWR45" H 1700 850 50  0001 C CNN
+F 0 "#PWR052" H 1700 850 50  0001 C CNN
 F 1 "VBUS" H 1700 1150 50  0000 C CNN
 F 2 "" H 1700 1000 50  0001 C CNN
@@
 $EndComp
 $Comp
-L VBUS #PWR48
+L VBUS #PWR053
 U 1 1 5A36EFB3
 P 2700 1400
-F 0 "#PWR48" H 2700 1250 50  0001 C CNN
+F 0 "#PWR053" H 2700 1250 50  0001 C CNN
 F 1 "VBUS" H 2700 1550 50  0000 C CNN
 F 2 "" H 2700 1400 50  0001 C CNN
@@
 NoConn ~ 3500 2900
 $Comp
-L +3.3V_FDTI #PWR50
+L +3.3V_FDTI #PWR054
 U 1 1 5A36F015
 P 2900 1300
-F 0 "#PWR50" H 2900 1150 50  0001 C CNN
+F 0 "#PWR054" H 2900 1150 50  0001 C CNN
 F 1 "+3.3V_FDTI" H 2900 1440 50  0000 C CNN
 F 2 "" H 2900 1300 50  0001 C CNN
@@
 DTR
 $Comp
-L GND #PWR43
+L GND #PWR055
 U 1 1 5A3703B4
 P 1300 1800
-F 0 "#PWR43" H 1300 1550 50  0001 C CNN
+F 0 "#PWR055" H 1300 1550 50  0001 C CNN
 F 1 "GND" H 1300 1650 50  0000 C CNN
 F 2 "" H 1300 1800 50  0001 C CNN
@@
 NoConn ~ 900  1300
 $Comp
-L GND #PWR42
+L GND #PWR056
 U 1 1 5A370474
 P 600 1050
-F 0 "#PWR42" H 600 800 50  0001 C CNN
+F 0 "#PWR056" H 600 800 50  0001 C CNN
 F 1 "GND" H 600 900 50  0000 C CNN
 F 2 "" H 600 1050 50  0001 C CNN

Commit message: Specified conda and resistors. PCB needs to be updated (usb condo from 1210 to 0805)
Parts:
- C10: footprint Capacitors_SMD:C_1210_HandSoldering -> Capacitors_SMD:C_0805_HandSoldering; symbol CP -> C; Manufacturer (none) -> Kemet; Manufacturer part number (none) -> C0805X475C4RACTU; Package (none) -> 0805
- C11, C13: Manufacturer (none) -> Kemet; Manufacturer part number (none) -> C0805X475C4RACTU; Package (none) -> 0805
- C12, C14: Manufacturer (none) -> Kemet; Manufacturer part number (none) -> C0805C104M3RACTU; Package (none) -> 0805
- J1: Manufacturer (none) -> Molex; Manufacturer part number (none) -> 47346-0001
- U6: Manufacturer (none) -> FTDI; Manufacturer part number (none) -> FT231XS-U; Package (none) -> SSOP-20
Changed lines of the file:
@@
 LIBS:freetronics_schematic
 LIBS:custom-power
-LIBS:74xgxx
-LIBS:74xx
-LIBS:ac-dc
-LIBS:actel
-LIBS:adc-dac
-LIBS:allegro
-LIBS:Altera
-LIBS:analog_devices
+LIBS:custom-charge
+LIBS:Amplifier_Audio
+LIBS:Amplifier_Buffer
+LIBS:Amplifier_Current
+LIBS:Amplifier_Difference
+LIBS:Amplifier_Instrumentation
+LIBS:Amplifier_Operational
+LIBS:Amplifier_Video
+LIBS:Analog
+LIBS:Analog_ADC
+LIBS:Analog_DAC
 LIBS:Analog_Switch
-LIBS:analog_switches
-LIBS:atmel
 LIBS:Audio
 LIBS:Battery_Management
-LIBS:bbd
-LIBS:bosch
-LIBS:brooktre
-LIBS:cmos_ieee
-LIBS:cmos4000
-LIBS:conn
+LIBS:Comparator
 LIBS:Connector_Generic
 LIBS:Connector_Generic_Shielded
 LIBS:Connector_Specialized
-LIBS:contrib
 LIBS:Converter_DCDC
 LIBS:CPLD_Altera
-LIBS:cypress
-LIBS:dc-dc
-LIBS:device
-LIBS:digital-audio
+LIBS:CPU
+LIBS:Device
 LIBS:Diode
-LIBS:display
+LIBS:Diode_Laser
 LIBS:Display_Character
 LIBS:Display_Graphic
@@
 LIBS:Driver_FET
 LIBS:Driver_LED
-LIBS:dsp
+LIBS:Driver_Motor
+LIBS:Driver_Relay
 LIBS:DSP_Freescale
 LIBS:DSP_Microchip_DSPIC33
 LIBS:DSP_Texas
-LIBS:elec-unifil
-LIBS:ESD_Protection
 LIBS:FPGA_Actel
-LIBS:ftdi
-LIBS:gennum
 LIBS:Graphic
-LIBS:hc11
-LIBS:intel
-LIBS:interface
+LIBS:Interface
 LIBS:Interface_CAN_LIN
+LIBS:Interface_CurrentLoop
 LIBS:Interface_Ethernet
+LIBS:Interface_Expansion
+LIBS:Interface_HID
+LIBS:Interface_LineDriver
+LIBS:Interface_Optical
 LIBS:Interface_Telecom
+LIBS:Interface_UART
 LIBS:Interface_USB
-LIBS:ir
-LIBS:Lattice
+LIBS:Isolator
+LIBS:Isolator_Analog
+LIBS:Jumper
 LIBS:LED
-LIBS:leds
-LIBS:linear
 LIBS:Logic_74xgxx
 LIBS:Logic_74xx
 LIBS:Logic_CMOS_4000
 LIBS:Logic_CMOS_IEEE
+LIBS:Logic_LevelTranslator
 LIBS:Logic_Programmable
 LIBS:Logic_TTL_IEEE
-LIBS:logo
-LIBS:maxim
 LIBS:MCU_AnalogDevices
+LIBS:MCU_Cypress
 LIBS:MCU_Infineon
 LIBS:MCU_Microchip_PIC10
@@
 LIBS:MCU_Microchip_PIC24
 LIBS:MCU_Microchip_PIC32
+LIBS:MCU_Microchip_SAME
+LIBS:MCU_Microchip_SAML
+LIBS:MCU_NXP_HC11
 LIBS:MCU_NXP_Kinetis
 LIBS:MCU_NXP_LPC
@@
 LIBS:MCU_ST_STM8
 LIBS:MCU_ST_STM32
+LIBS:MCU_Texas
 LIBS:MCU_Texas_MSP430
 LIBS:Mechanical
-LIBS:memory
+LIBS:Memory_Controller
 LIBS:Memory_EEPROM
 LIBS:Memory_Flash
 LIBS:Memory_NVRAM
 LIBS:Memory_RAM
-LIBS:microchip
-LIBS:microchip_dspic33dsc
-LIBS:microchip_pic10mcu
-LIBS:microchip_pic12mcu
-LIBS:microchip_pic16mcu
-LIBS:microchip_pic18mcu
-LIBS:microchip_pic24mcu
-LIBS:microchip_pic32mcu
-LIBS:microcontrollers
-LIBS:modules
+LIBS:Memory_UniqueID
 LIBS:Motor
-LIBS:motor_drivers
-LIBS:motorola
-LIBS:motors
-LIBS:msp430
-LIBS:nordicsemi
-LIBS:nxp
-LIBS:nxp_armmcu
-LIBS:onsemi
-LIBS:opto
 LIBS:Oscillator
-LIBS:Oscillators
-LIBS:philips
 LIBS:Potentiometer_Digital
 LIBS:power
 LIBS:Power_Management
 LIBS:Power_Protection
-LIBS:powerint
+LIBS:Power_Supervisor
 LIBS:pspice
 LIBS:Reference_Current
 LIBS:Reference_Voltage
-LIBS:references
-LIBS:regul
 LIBS:Regulator_Controller
 LIBS:Regulator_Current
@@
 LIBS:Regulator_Switching
 LIBS:Relay
-LIBS:relays
+LIBS:Relay_SolidState
 LIBS:RF_AM_FM
 LIBS:RF_Bluetooth
+LIBS:RF_Mixer
 LIBS:RF_Module
+LIBS:RF_RFID
 LIBS:RF_WiFi
-LIBS:rfcom
 LIBS:Sensor
 LIBS:Sensor_Audio
@@
 LIBS:Sensor_Optical
 LIBS:Sensor_Pressure
+LIBS:Sensor_Proximity
 LIBS:Sensor_Temperature
 LIBS:Sensor_Touch
 LIBS:Sensor_Voltage
-LIBS:sensors
-LIBS:silabs
-LIBS:siliconi
-LIBS:stm8
-LIBS:stm32
-LIBS:supertex
 LIBS:Switch
-LIBS:switches
-LIBS:texas
 LIBS:Timer
-LIBS:transf
+LIBS:Timer_RTC
 LIBS:Transformer
+LIBS:Transistor_Array
 LIBS:Transistor_BJT
 LIBS:Transistor_FET
 LIBS:Transistor_IGBT
-LIBS:transistors
-LIBS:triac_thyristor
-LIBS:ttl_ieee
 LIBS:Valve
-LIBS:valves
-LIBS:video
-LIBS:wiznet
-LIBS:Worldsemi
-LIBS:Xicor
-LIBS:xilinx
-LIBS:zetex
-LIBS:Zilog
-LIBS:custom-charge
+LIBS:Video
 LIBS:gpstracker-cache
 EELAYER 25 0
@@
 F 2 "Housings_SSOP:SSOP-20_4.4x6.5mm_Pitch0.65mm" H 2800 2300 50  0001 C CNN
 F 3 "" H 2800 2300 50  0001 C CNN
+F 4 "FTDI" H 2800 2300 60  0001 C CNN "Manufacturer"
+F 5 "FT231XS-U" H 2800 2300 60  0001 C CNN "Manufacturer part number"
+F 6 "SSOP-20" H 2800 2300 60  0001 C CNN "Package"
 	1    2800 2300
 	1    0    0    -1
@@
 F 2 "Capacitors_SMD:C_0805_HandSoldering" H 2038 2400 50  0001 C CNN
 F 3 "" H 2000 2550 50  0001 C CNN
+F 4 "Kemet" H 2000 2550 60  0001 C CNN "Manufacturer"
+F 5 "C0805C104M3RACTU" H 2000 2550 60  0001 C CNN "Manufacturer part number"
+F 6 "0805" H 2000 2550 60  0001 C CNN "Package"
 	1    2000 2550
 	1    0    0    -1
@@
 F 2 "Capacitors_SMD:C_0805_HandSoldering" H 1388 2150 50  0001 C CNN
 F 3 "" H 1350 2300 50  0001 C CNN
+F 4 "Kemet" H 1350 2300 60  0001 C CNN "Manufacturer"
+F 5 "C0805X475C4RACTU" H 1350 2300 60  0001 C CNN "Manufacturer part number"
+F 6 "0805" H 1350 2300 60  0001 C CNN "Package"
 	1    1350 2300
 	1    0    0    -1
@@
 F 2 "Capacitors_SMD:C_0805_HandSoldering" H 1638 1400 50  0001 C CNN
 F 3 "" H 1600 1550 50  0001 C CNN
+F 4 "Kemet" H 1600 1550 60  0001 C CNN "Manufacturer"
+F 5 "C0805C104M3RACTU" H 1600 1550 60  0001 C CNN "Manufacturer part number"
+F 6 "0805" H 1600 1550 60  0001 C CNN "Package"
 	1    1600 1550
 	1    0    0    -1
@@
 F 2 "Capacitors_SMD:C_0805_HandSoldering" H 1038 2150 50  0001 C CNN
 F 3 "" H 1000 2300 50  0001 C CNN
+F 4 "Kemet" H 1000 2300 60  0001 C CNN "Manufacturer"
+F 5 "C0805X475C4RACTU" H 1000 2300 60  0001 C CNN "Manufacturer part number"
+F 6 "0805" H 1000 2300 60  0001 C CNN "Package"
 	1    1000 2300
 	1    0    0    -1
@@
 F 2 "Connectors_USB:USB_Micro-B_Molex_47346-0001" H 1250 950 50  0001 C CNN
 F 3 "" H 1250 950 50  0001 C CNN
+F 4 "Molex" H 1100 1000 60  0001 C CNN "Manufacturer"
+F 5 "47346-0001" H 1100 1000 60  0001 C CNN "Manufacturer part number"
 	1    1100 1000
 	0    1    1    0
@@
 Connection ~ 1300 1350
 $Comp
-L CP C10
+L C C10
 U 1 1 5A371566
 P 1300 1550
 F 0 "C10" H 1325 1650 50  0000 L CNN
 F 1 "4.7uF" H 1325 1450 50  0000 L CNN
-F 2 "Capacitors_SMD:C_1210_HandSoldering" H 1338 1400 50  0001 C CNN
+F 2 "Capacitors_SMD:C_0805_HandSoldering" H 1338 1400 50  0001 C CNN
 F 3 "" H 1300 1550 50  0001 C CNN
+F 4 "Kemet" H 1300 1550 60  0001 C CNN "Manufacturer"
+F 5 "C0805X475C4RACTU" H 1300 1550 60  0001 C CNN "Manufacturer part number"
+F 6 "0805" H 1300 1550 60  0001 C CNN "Package"
 	1    1300 1550
 	1    0    0    -1

Commit message: Made the usb connector vertical
Parts:
- J1: footprint Connectors_USB:USB_Micro-B_Molex_47346-0001 -> Connectors_USB:USB_Micro-B_Vertical_Molex-105133-0001
Changed lines of the file:
@@
 F 0 "J1" H 900 1450 50  0000 L CNN
 F 1 "Molex 47346-0001" H 900 1350 50  0001 L CNN
-F 2 "Connectors_USB:USB_Micro-B_Molex_47346-0001" H 1250 950 50  0001 C CNN
+F 2 "Connectors_USB:USB_Micro-B_Vertical_Molex-105133-0001" H 1250 950 50  0001 C CNN
 F 3 "" H 1250 950 50  0001 C CNN
 F 4 "Molex" H 1100 1000 60  0001 C CNN "Manufacturer"

Commit message: Ordered PCB
Parts:
- J1: value Molex 47346-0001 -> Molex 105133-0002; footprint Connectors_USB:USB_Micro-B_Vertical_Molex-105133-0001 -> custom-conn:USB_Micro-B_Vertical_Molex-105133-0001_HandSoldering; Manufacturer part number 47346-0001 -> 105133-0002
- LED6: Manufacturer (none) -> Kingbright; Manufacturer part number (none) -> APT2012SYCK; Package (none) -> 0805
- LED7: Manufacturer (none) -> Kingbright; Manufacturer part number (none) -> APT2012EC; Package (none) -> 0805
- R16, R17: Manufacturer (none) -> Panasonic; Manufacturer part number (none) -> ERJ-6GEYJ270V; Package (none) -> 0805
- R18, R19: Manufacturer (none) -> Panasonic; Manufacturer part number (none) -> ERJ-6GEYJ102V; Package (none) -> 0805
Connections:
- net +3V3_FDTI: now also C12.1, U6.14 (~RESET)
Changed lines of the file:
@@
-$EndComp
-$Comp
-L R R19
-U 1 1 5A368449
-P 4450 2400
-F 0 "R19" V 4530 2400 50  0000 C CNN
-F 1 "1k" V 4450 2400 50  0000 C CNN
-F 2 "Resistors_SMD:R_0805_HandSoldering" H 4450 2400 60  0001 C CNN
-F 3 "" H 4450 2400 60  0000 C CNN
-	1    4450 2400
-	-1   0    0    1
 $EndComp
 $Comp
@@
 F 2 "Resistors_SMD:R_0805_HandSoldering" H 4150 2400 60  0001 C CNN
 F 3 "" H 4150 2400 60  0000 C CNN
+F 4 "Panasonic" V 4150 2400 60  0001 C CNN "Manufacturer"
+F 5 "ERJ-6GEYJ102V" V 4150 2400 60  0001 C CNN "Manufacturer part number"
+F 6 "0805" V 4150 2400 60  0001 C CNN "Package"
 	1    4150 2400
 	-1   0    0    1
@@
 $EndComp
 $Comp
-L R R17
-U 1 1 5A36872C
-P 1850 2000
-F 0 "R17" V 1950 2000 50  0000 C CNN
-F 1 "27R" V 1850 2000 50  0000 C CNN
-F 2 "Resistors_SMD:R_0805_HandSoldering" H 1850 2000 60  0001 C CNN
-F 3 "" H 1850 2000 60  0000 C CNN
-	1    1850 2000
-	0    -1   -1   0
-$EndComp
-$Comp
 L R R16
 U 1 1 5A36875E
@@
 F 2 "Resistors_SMD:R_0805_HandSoldering" H 1850 2100 60  0001 C CNN
 F 3 "" H 1850 2100 60  0000 C CNN
+F 4 "Panasonic" V 1850 2100 60  0001 C CNN "Manufacturer"
+F 5 "ERJ-6GEYJ270V" V 1850 2100 60  0001 C CNN "Manufacturer part number"
+F 6 "0805" V 1850 2100 60  0001 C CNN "Package"
 	1    1850 2100
 	0    1    1    0
@@
 F 2 "LEDs:LED_0805_HandSoldering" H 4150 2000 60  0001 C CNN
 F 3 "" H 4150 2000 60  0000 C CNN
+F 4 "Kingbright" H 4150 2000 60  0001 C CNN "Manufacturer"
+F 5 "APT2012SYCK" H 4150 2000 60  0001 C CNN "Manufacturer part number"
+F 6 "0805" H 4150 2000 60  0001 C CNN "Package"
 	1    4150 2000
 	0    1    1    0
@@
 F 2 "LEDs:LED_0805_HandSoldering" H 4450 2000 60  0001 C CNN
 F 3 "" H 4450 2000 60  0000 C CNN
+F 4 "Kingbright" H 4450 2000 60  0001 C CNN "Manufacturer"
+F 5 "APT2012EC" H 4450 2000 60  0001 C CNN "Manufacturer part number"
+F 6 "0805" H 4450 2000 60  0001 C CNN "Package"
 	1    4450 2000
 	0    1    1    0
@@
 P 1100 1000
 F 0 "J1" H 900 1450 50  0000 L CNN
-F 1 "Molex 47346-0001" H 900 1350 50  0001 L CNN
-F 2 "Connectors_USB:USB_Micro-B_Vertical_Molex-105133-0001" H 1250 950 50  0001 C CNN
+F 1 "Molex 105133-0002" H 900 1350 50  0001 L CNN
+F 2 "custom-conn:USB_Micro-B_Vertical_Molex-105133-0001_HandSoldering" H 1250 950 50  0001 C CNN
 F 3 "" H 1250 950 50  0001 C CNN
 F 4 "Molex" H 1100 1000 60  0001 C CNN "Manufacturer"
-F 5 "47346-0001" H 1100 1000 60  0001 C CNN "Manufacturer part number"
+F 5 "105133-0002" H 1100 1000 60  0001 C CNN "Manufacturer part number"
 	1    1100 1000
 	0    1    1    0
@@
 	2050 1700 2100 1700
 Wire Wire Line
-	2050 1700 2050 1650
+	2050 1650 2050 2300
 Wire Wire Line
 	4150 1850 4150 1800
@@
 Text Notes 2300 900  0    120  ~ 24
 USB Interface
+$Comp
+L R R19
+U 1 1 5A52C333
+P 4450 2400
+F 0 "R19" V 4530 2400 50  0000 C CNN
+F 1 "1k" V 4450 2400 50  0000 C CNN
+F 2 "Resistors_SMD:R_0805_HandSoldering" H 4450 2400 60  0001 C CNN
+F 3 "" H 4450 2400 60  0000 C CNN
+F 4 "Panasonic" V 4450 2400 60  0001 C CNN "Manufacturer"
+F 5 "ERJ-6GEYJ102V" V 4450 2400 60  0001 C CNN "Manufacturer part number"
+F 6 "0805" V 4450 2400 60  0001 C CNN "Package"
+	1    4450 2400
+	-1   0    0    1
+$EndComp
+$Comp
+L R R17
+U 1 1 5A534FBA
+P 1850 2000
+F 0 "R17" V 1950 2000 50  0000 C CNN
+F 1 "27R" V 1850 2000 50  0000 C CNN
+F 2 "Resistors_SMD:R_0805_HandSoldering" H 1850 2000 60  0001 C CNN
+F 3 "" H 1850 2000 60  0000 C CNN
+F 4 "Panasonic" V 1850 2000 60  0001 C CNN "Manufacturer"
+F 5 "ERJ-6GEYJ270V" V 1850 2000 60  0001 C CNN "Manufacturer part number"
+F 6 "0805" V 1850 2000 60  0001 C CNN "Package"
+	1    1850 2000
+	0    -1   -1   0
+$EndComp
+Connection ~ 2050 2300
+Connection ~ 2050 1700
 $EndSCHEMATC
