File: gpstracker.kicad_pcb (KiCad board)
At the start: 2 copper layers, 75.2 x 54.6 mm, 185 parts, among them IC1 SIM808, J1 Molex 105133-0002, J2 Leds, J3 47553-0001, J4 CONN_COAXIAL, J5 CONN_COAXIAL, J6 Micro_SD_Card, Q1 DMP1045U, SW1 Reset, U1 MCP73832-5-OT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

Commit message: Ordered PCB
Parts:
- removed the REF** at (171.2, 118.4)
- removed the REF** at (171.2, 73.4)
- removed the REF** at (105.7, 118.4)
- removed the VIA** at (145.8, 122.4)
- removed the VIA** at (138.4, 122.4)
- removed the VIA** at (131.1, 122.4)
- removed the VIA** at (123.7, 122.4)
- removed the VIA** at (116.3, 122.4)
- removed the VIA** at (109.0, 122.4)
- removed the VIA** at (101.6, 122.4)
- removed the VIA** at (175.3, 117.1)
- removed the VIA** at (175.3, 111.8)
- removed the VIA** at (175.3, 106.5)
- removed the VIA** at (175.3, 101.2)
- removed the VIA** at (175.3, 95.9)
- removed the VIA** at (175.3, 90.6)
- removed the VIA** at (175.3, 85.3)
- removed the VIA** at (175.3, 80.0)
- removed the VIA** at (175.3, 74.7)
- removed the VIA** at (175.3, 69.3)
- removed the VIA** at (167.9, 69.3)
- removed the VIA** at (160.5, 69.3)
- removed the VIA** at (153.2, 69.3)
- removed the VIA** at (145.8, 69.3)
- removed the VIA** at (138.4, 69.3)
- removed the VIA** at (131.1, 69.3)
- removed the VIA** at (123.7, 69.3)
- removed the VIA** at (116.3, 69.3)
- removed the VIA** at (109.0, 69.3)
- removed the VIA** at (101.6, 74.7)
- removed the VIA** at (101.6, 80.0)
- removed the VIA** at (101.6, 85.3)
- removed the VIA** at (101.6, 90.6)
- removed the VIA** at (101.6, 95.9)
- removed the VIA** at (101.6, 101.2)
- removed the VIA** at (101.6, 106.5)
- removed the VIA** at (101.6, 111.8)
- removed the VIA** at (101.6, 117.1)
- removed the VIA** at (175.3, 122.4)
- removed the VIA** at (167.9, 122.4)
- removed the VIA** at (160.5, 122.4)
- removed the VIA** at (153.2, 122.4)
- added REF**: MountingHole_3.2mm_M3_Pad, Mounting_Holes:MountingHole_3.2mm_M3_Pad, F.Cu at (173.9, 123.4)
- added REF**: MountingHole_3.2mm_M3_Pad, Mounting_Holes:MountingHole_3.2mm_M3_Pad, F.Cu at (103.9, 123.4)
- added REF**: MountingHole_3.2mm_M3_Pad, Mounting_Holes:MountingHole_3.2mm_M3_Pad, F.Cu at (173.9, 73.4)
- added VIA**: Via-0.6mm, custom-conn:Via-0.6mm, F.Cu at (175.0, 101.1)
- added VIA**: Via-0.6mm, custom-conn:Via-0.6mm, F.Cu at (177.8, 110.0)
- added VIA**: Via-0.6mm, custom-conn:Via-0.6mm, F.Cu at (177.8, 104.2)
- added VIA**: Via-0.6mm, custom-conn:Via-0.6mm, F.Cu at (177.8, 98.4)
- added VIA**: Via-0.6mm, custom-conn:Via-0.6mm, F.Cu at (177.8, 92.7)
- added VIA**: Via-0.6mm, custom-conn:Via-0.6mm, F.Cu at (177.8, 86.9)
- added VIA**: Via-0.6mm, custom-conn:Via-0.6mm, F.Cu at (177.8, 81.1)
- added VIA**: Via-0.6mm, custom-conn:Via-0.6mm, F.Cu at (177.8, 75.4)
- added VIA** (x2): Via-0.6mm, custom-conn:Via-0.6mm, F.Cu at (177.8, 127.3)
- added VIA**: Via-0.6mm, custom-conn:Via-0.6mm, F.Cu at (170.0, 127.3)
- added VIA**: Via-0.6mm, custom-conn:Via-0.6mm, F.Cu at (162.3, 127.3)
- added VIA**: Via-0.6mm, custom-conn:Via-0.6mm, F.Cu at (164.4, 122.7)
- added VIA**: Via-0.6mm, custom-conn:Via-0.6mm, F.Cu at (154.5, 127.3)
- added VIA**: Via-0.6mm, custom-conn:Via-0.6mm, F.Cu at (146.7, 127.3)
- added VIA**: Via-0.6mm, custom-conn:Via-0.6mm, F.Cu at (138.9, 127.3)
- added VIA**: Via-0.6mm, custom-conn:Via-0.6mm, F.Cu at (131.2, 127.3)
- added VIA**: Via-0.6mm, custom-conn:Via-0.6mm, F.Cu at (123.4, 127.3)
- added VIA**: Via-0.6mm, custom-conn:Via-0.6mm, F.Cu at (115.6, 127.3)
- added VIA**: Via-0.6mm, custom-conn:Via-0.6mm, F.Cu at (107.8, 127.3)
- added VIA**: Via-0.6mm, custom-conn:Via-0.6mm, F.Cu at (100.1, 127.3)
- added VIA**: Via-0.6mm, custom-conn:Via-0.6mm, F.Cu at (100.1, 121.5)
- added VIA**: Via-0.6mm, custom-conn:Via-0.6mm, F.Cu at (100.1, 115.7)
- added VIA**: Via-0.6mm, custom-conn:Via-0.6mm, F.Cu at (140.0, 122.7)
- added VIA**: Via-0.6mm, custom-conn:Via-0.6mm, F.Cu at (100.1, 110.0)
- added VIA**: Via-0.6mm, custom-conn:Via-0.6mm, F.Cu at (100.1, 104.2)
- added VIA**: Via-0.6mm, custom-conn:Via-0.6mm, F.Cu at (100.1, 98.4)
- added VIA**: Via-0.6mm, custom-conn:Via-0.6mm, F.Cu at (100.1, 92.7)
- added VIA**: Via-0.6mm, custom-conn:Via-0.6mm, F.Cu at (100.1, 86.9)
- added VIA**: Via-0.6mm, custom-conn:Via-0.6mm, F.Cu at (100.1, 81.1)
- added VIA**: Via-0.6mm, custom-conn:Via-0.6mm, F.Cu at (100.1, 75.4)
- added VIA**: Via-0.6mm, custom-conn:Via-0.6mm, F.Cu at (177.8, 69.6)
- added VIA**: Via-0.6mm, custom-conn:Via-0.6mm, F.Cu at (170.0, 69.6)
- added VIA**: Via-0.6mm, custom-conn:Via-0.6mm, F.Cu at (162.3, 69.6)
- added VIA**: Via-0.6mm, custom-conn:Via-0.6mm, F.Cu at (119.4, 122.4)
- added VIA**: Via-0.6mm, custom-conn:Via-0.6mm, F.Cu at (154.5, 69.6)
- added VIA**: Via-0.6mm, custom-conn:Via-0.6mm, F.Cu at (146.7, 69.6)
- added VIA**: Via-0.6mm, custom-conn:Via-0.6mm, F.Cu at (138.9, 69.6)
- added VIA**: Via-0.6mm, custom-conn:Via-0.6mm, F.Cu at (131.2, 69.6)
- added VIA**: Via-0.6mm, custom-conn:Via-0.6mm, F.Cu at (123.4, 69.6)
- added VIA**: Via-0.6mm, custom-conn:Via-0.6mm, F.Cu at (115.6, 69.6)
- added VIA**: Via-0.6mm, custom-conn:Via-0.6mm, F.Cu at (107.8, 69.6)
- added VIA**: Via-0.6mm, custom-conn:Via-0.6mm, F.Cu at (113.6, 122.4)
- added VIA**: Via-0.6mm, custom-conn:Via-0.6mm, F.Cu at (175.0, 111.8)
- added VIA**: Via-0.6mm, custom-conn:Via-0.6mm, F.Cu at (177.8, 121.5)
- added VIA**: Via-0.6mm, custom-conn:Via-0.6mm, F.Cu at (177.8, 115.7)
- R14, R15: value 50k -> 51k
- R3: value 470R -> 1k
- SW1: footprint Buttons_Switches_SMD:SW_SPST_EVPBF -> Buttons_Switches_SMD:SW_SPST_B3S-1000
- moved J2 10.2 mm to (149.4, 123.4)
- moved REF** 1.78 mm to (103.9, 73.4)
- moved VIA** 1.55 mm to (100.1, 69.6)
- moved C5 1.37 mm to (122.7, 119.4)
- moved R6 1.37 mm to (124.7, 119.4)
- moved SW1 0.51 mm to (130.8, 118.9)
- moved VIA** 0.38 mm to (170.9, 103.6)
- moved VIA** 0.25 mm to (121.5, 93.0)
Connections:
- C12 pad 1: Net-(C12-Pad1) -> +3V3_FDTI
- REF** pad 1: GND -> (no net)
- U6 pad 14: Net-(C12-Pad1) -> +3V3_FDTI
Routing:
- net +3V3_FDTI: track 20.5 -> 24.7 mm
- net Net-(C12-Pad1): track 3.55 -> 0.00 mm
- net /DTR: track 20.8 -> 22.3 mm
- net +3V3: track 123.8 -> 125.3 mm
- net GND: track 34.6 -> 35.7 mm
- net /ARD_RST: track 60.8 -> 61.8 mm
Other:
- board outline removed
